File: Core-SensorTH/Core-SensorTH.kicad_pcb (KiCad board)
At the start: 2 copper layers, 23 x 14 mm, 13 parts, among them J1 PH-4AW, Q1 CJ2102, Q2 CJ2102, U1 HX9193-33GB, U2 AHT10

Commit message: 增加接口丝印标识
Signed-off-by: fuhua-chen <fuhua-chen@outlook.com>
Other:
- board text added: "GND"
- board text added: "SCL"
- board text added: "SDA"
- board text added: "VCC"
Changed lines of the file:
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@@
   (general
     (thickness 1.6)
-    (drawings 29)
+    (drawings 33)
     (tracks 105)
     (zones 0)
@@
     (pad_to_mask_clearance 0)
     (aux_axis_origin 0 0)
-    (visible_elements FFFFFF7F)
+    (visible_elements 7FFFFFFF)
     (pcbplotparams
       (layerselection 0x010fc_ffffffff)
@@
       (drillshape 0)
       (scaleselection 1)
-      (outputdirectory "Core-SensorTH v0.1"))
+      (outputdirectory "Core-SensorTH v0.1-Gerber"))
   )
   (net 0 "")
@@
     (pad 6 smd rect (at 1.6 -1.27) (size 1.27 1) (layers F.Cu F.Paste F.Mask))
   )
+  (gr_text SCL (at 132.68 105.05) (layer B.SilkS)
+    (effects (font (size 0.8 0.8) (thickness 0.152)) (justify mirror))
+  )
+  (gr_text SDA (at 132.6 103.01) (layer B.SilkS)
+    (effects (font (size 0.8 0.8) (thickness 0.152)) (justify mirror))
+  )
+  (gr_text VCC (at 132.68 101) (layer B.SilkS)
+    (effects (font (size 0.8 0.8) (thickness 0.152)) (justify mirror))
+  )
+  (gr_text GND (at 132.68 99.07) (layer B.SilkS)
+    (effects (font (size 0.8 0.8) (thickness 0.152)) (justify mirror))
+  )
   (gr_text "CoreSensorTH\nv0.1 20200301" (at 142.87 101.62 90) (layer B.SilkS)
